Commit message: changing the size of the rocket for better simulation

File: assets/landing_pad.urdf (robot description, URDF)
Before this commit: robot landing_pad, 1 links, 0 joints
Links:
- link pad: geometry collision cylinder length=0.1 radius=10; visual cylinder length=0.1 radius=10

File: assets/rocket.urdf (robot description, URDF)
Before this commit: robot falcon9, 5 links, 4 joints
Links:
- link body: geometry collision cylinder length=14 radius=1.0; visual cylinder length=14 radius=1.0
- link leg1: geometry collision box size=3.5 0.5 0.5; visual box size=3.5 0.5 0.5
- link leg2: geometry collision box size=3.5 0.5 0.5; visual box size=3.5 0.5 0.5
- link leg3: geometry collision box size=3.5 0.5 0.5; visual box size=3.5 0.5 0.5
- link leg4: geometry collision box size=3.5 0.5 0.5; visual box size=3.5 0.5 0.5
Joints:
- joint leg1_joint: origin xyz=0.3 0 -1.83 rpy=0 0.8 0 -> xyz=1.0 0 -6.69 rpy=0 0.8 0
- joint leg2_joint: origin xyz=-0.3 0 -1.83 rpy=0 -0.8 0 -> xyz=-1.0 0 -6.69 rpy=0 -0.8 0
- joint leg3_joint: origin xyz=0 0.3 -1.83 rpy=0 0.8 1.57 -> xyz=0 1 -6.69 rpy=0 0.8 1.57
- joint leg4_joint: origin xyz=0 -0.3 -1.83 rpy=0 -0.8 1.57 -> xyz=0 -1 -6.69 rpy=0 -0.8 1.57

Commit message: Revert "changing the size of the rocket for better simulation"
This reverts commit e2c6ad4fc9031b4e423389c36bcc8c7d831dddcb.

File: assets/landing_pad.urdf (robot description, URDF)
Before this commit: robot landing_pad, 1 links, 0 joints
Links:
- link pad: geometry collision cylinder length=0.1 radius=10; visual cylinder length=0.1 radius=5

File: assets/rocket.urdf (robot description, URDF)
Before this commit: robot falcon9, 5 links, 4 joints
Links:
- link body: geometry collision cylinder length=3.8 radius=0.3; visual cylinder length=3.8 radius=0.3
- link leg1: geometry collision box size=1.2 0.15 0.07; visual box size=1.2 0.15 0.07
- link leg2: geometry collision box size=1.2 0.15 0.07; visual box size=1.2 0.15 0.07
- link leg3: geometry collision box size=1.2 0.15 0.07; visual box size=1.2 0.15 0.07
- link leg4: geometry collision box size=1.2 0.15 0.07; visual box size=1.2 0.15 0.07
Joints:
- joint leg1_joint: origin xyz=1.0 0 -6.69 rpy=0 0.8 0 -> xyz=0.3 0 -1.83 rpy=0 0.8 0
- joint leg2_joint: origin xyz=-1.0 0 -6.69 rpy=0 -0.8 0 -> xyz=-0.3 0 -1.83 rpy=0 -0.8 0
- joint leg3_joint: origin xyz=0 1 -6.69 rpy=0 0.8 1.57 -> xyz=0 0.3 -1.83 rpy=0 0.8 1.57
- joint leg4_joint: origin xyz=0 -1 -6.69 rpy=0 -0.8 1.57 -> xyz=0 -0.3 -1.83 rpy=0 -0.8 1.57

Commit message: changing the parmeter according to the size of the rocket

File: assets/landing_pad.urdf (robot description, URDF)
Before this commit: robot landing_pad, 1 links, 0 joints
Links:
- link pad: geometry collision cylinder length=0.1 radius=20; visual cylinder length=0.1 radius=20

Commit message: adding 'how to install section' in readme

File: assets/landing_pad.urdf (robot description, URDF)
Before this commit: robot landing_pad, 1 links, 0 joints
Links:
- link pad: geometry collision cylinder length=0.1 radius=10; visual cylinder length=0.1 radius=7
